File: rj12-breakout-bb.kicad_sch (KiCad schematic)
At the start: 0 parts

Commit message: Initial version
Parts:
- added J1: RJ12, Connector_RJ:RJ12_Amphenol_54601, symbol Chof747 Connectors:RJ12
- added J2: Front, Connector_PinHeader_2.54mm:PinHeader_1x04_P2.54mm_Vertical, symbol Connector:Conn_01x04_Pin
- added J3: Back, Connector_PinHeader_2.54mm:PinHeader_1x04_P2.54mm_Vertical, symbol Connector:Conn_01x04_Pin
Connections:
- new net: J1.5, J2.1 (Pin_1), J3.1 (Pin_1)
- new net: J1.2, J2.2 (Pin_2), J3.2 (Pin_2)
- new net: J1.3, J2.3 (Pin_3), J3.3 (Pin_3)
- new net: J1.4, J2.4 (Pin_4), J3.4 (Pin_4)
Other:
- title: (none) -> RJ12 Breakout Board for Breadboards
Changed lines of the file:
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@@
 (kicad_sch (version 20230121) (generator eeschema)
-  (paper "A4")
+  (paper "A5")
   (title_block
+    (title "RJ12 Breakout Board for Breadboards")
     (company "chof.org")
   )
+  (junction (at 106.68 44.45) (diameter 0) (color 0 0 0 0)
+  )
+  (junction (at 107.95 46.99) (diameter 0) (color 0 0 0 0)
+  )
+  (junction (at 109.22 49.53) (diameter 0) (color 0 0 0 0)
+  )
+  (junction (at 110.49 52.07) (diameter 0) (color 0 0 0 0)
+  )
+  (wire (pts (xy 110.49 69.85) (xy 123.19 69.85))
+    (stroke (width 0) (type default))
+  )
+  (wire (pts (xy 107.95 46.99) (xy 107.95 64.77))
+    (stroke (width 0) (type default))
+  )
+  (wire (pts (xy 109.22 49.53) (xy 123.19 49.53))
+    (stroke (width 0) (type default))
+  )
+  (wire (pts (xy 102.87 52.07) (xy 110.49 52.07))
+    (stroke (width 0) (type default))
+  )
+  (wire (pts (xy 110.49 52.07) (xy 123.19 52.07))
+    (stroke (width 0) (type default))
+  )
+  (wire (pts (xy 107.95 64.77) (xy 123.19 64.77))
+    (stroke (width 0) (type default))
+  )
+  (wire (pts (xy 110.49 52.07) (xy 110.49 69.85))
+    (stroke (width 0) (type default))
+  )
+  (wire (pts (xy 107.95 46.99) (xy 123.19 46.99))
+    (stroke (width 0) (type default))
+  )
+  (wire (pts (xy 102.87 46.99) (xy 107.95 46.99))
+    (stroke (width 0) (type default))
+  )
+  (wire (pts (xy 106.68 62.23) (xy 123.19 62.23))
+    (stroke (width 0) (type default))
+  )
+  (wire (pts (xy 109.22 49.53) (xy 109.22 67.31))
+    (stroke (width 0) (type default))
+  )
+  (wire (pts (xy 106.68 44.45) (xy 106.68 62.23))
+    (stroke (width 0) (type default))
+  )
+  (wire (pts (xy 106.68 44.45) (xy 123.19 44.45))
+    (stroke (width 0) (type default))
+  )
+  (wire (pts (xy 109.22 67.31) (xy 123.19 67.31))
+    (stroke (width 0) (type default))
+  )
+  (wire (pts (xy 102.87 44.45) (xy 106.68 44.45))
+    (stroke (width 0) (type default))
+  )
+  (wire (pts (xy 102.87 49.53) (xy 109.22 49.53))
+    (stroke (width 0) (type default))
+  )
+  (symbol (lib_id "Connector:Conn_01x04_Pin") (at 128.27 49.53 180) (unit 1)
+    (in_bom yes) (on_board yes) (dnp no)
+    (property "Reference" "J2" (at 127.635 55.88 0)
+      (effects (font (size 1.27 1.27)))
+    )
+    (property "Value" "Front" (at 127.635 53.34 0)
+      (effects (font (size 1.27 1.27)))
+    )
+    (property "Footprint" "Connector_PinHeader_2.54mm:PinHeader_1x04_P2.54mm_Vertical" (at 128.27 49.53 0)
+      (effects (font (size 1.27 1.27)) hide)
+    )
+    (property "Datasheet" "~" (at 128.27 49.53 0)
+      (effects (font (size 1.27 1.27)) hide)
+    )
+    (pin "1")
+    (pin "2")
+    (pin "3")
+    (pin "4")
+    (instances
+      (project "rj12-breakout-bb"
+        (path "/e8426e51-e5a9-4642-8277-6d3f50e0e523"
+          (reference "J2") (unit 1)
+        )
+      )
+    )
+  )
+  (symbol (lib_id "Connector:Conn_01x04_Pin") (at 128.27 67.31 180) (unit 1)
+    (in_bom yes) (on_board yes) (dnp no)
+    (property "Reference" "J3" (at 127.635 73.66 0)
+      (effects (font (size 1.27 1.27)))
+    )
+    (property "Value" "Back" (at 127.635 71.12 0)
+      (effects (font (size 1.27 1.27)))
+    )
+    (property "Footprint" "Connector_PinHeader_2.54mm:PinHeader_1x04_P2.54mm_Vertical" (at 128.27 67.31 0)
+      (effects (font (size 1.27 1.27)) hide)
+    )
+    (property "Datasheet" "~" (at 128.27 67.31 0)
+      (effects (font (size 1.27 1.27)) hide)
+    )
+    (pin "1")
+    (pin "2")
+    (pin "3")
+    (pin "4")
+    (instances
+      (project "rj12-breakout-bb"
+        (path "/e8426e51-e5a9-4642-8277-6d3f50e0e523"
+          (reference "J3") (unit 1)
+        )
+      )
+    )
+  )
+  (symbol (lib_id "Chof747 Connectors:RJ12") (at 92.71 49.53 0) (unit 1)
+    (in_bom yes) (on_board yes) (dnp no) (fields_autoplaced)
+    (property "Reference" "J1" (at 92.71 38.1 0)
+      (effects (font (size 1.27 1.27)))
+    )
+    (property "Value" "RJ12" (at 92.71 40.64 0)
+      (effects (font (size 1.27 1.27)))
+    )
+    (property "Footprint" "Connector_RJ:RJ12_Amphenol_54601" (at 92.71 48.26 90)
+      (effects (font (size 1.27 1.27)) hide)
+    )
+    (property "Datasheet" "~" (at 92.71 48.26 90)
+      (effects (font (size 1.27 1.27)) hide)
+    )
+    (pin "2")
+    (pin "3")
+    (pin "4")
+    (pin "5")
+    (instances
+      (project "rj12-breakout-bb"
+        (path "/e8426e51-e5a9-4642-8277-6d3f50e0e523"
+          (reference "J1") (unit 1)
+        )
+      )
+    )
+  )
   (sheet_instances
