File: rj12-breakout-bb.kicad_pcb (KiCad board)
At the start: 2 copper layers, 2 parts

Commit message: Initial version
Parts:
- removed the G*** at (22.4, 182.3)
- added J1: RJ12, Connector_RJ:RJ12_Amphenol_54601, F.Cu at (110.8, 73.9)
- added J2: Front, Connector_PinHeader_2.54mm:PinHeader_1x04_P2.54mm_Vertical, B.Cu at (116.8, 80.9)
- added J3: Back, Connector_PinHeader_2.54mm:PinHeader_1x04_P2.54mm_Vertical, B.Cu at (124.5, 80.9)
- moved G*** 126.7 mm to (97.6, 77.4)
Routing:
- net Net-(J2-Pin_4): track 0.00 -> 23.2 mm
- net Net-(J2-Pin_2): track 0.00 -> 18.0 mm
- net Net-(J2-Pin_1): track 0.00 -> 14.4 mm
- net Net-(J2-Pin_3): track 0.00 -> 13.9 mm
Other:
- board outline added: 32.3 x 14.6 mm
- board text added: "2"
- board text added: "3"
- board text added: "4"
- board text added: "5"
- board text added: "RJ12 BB v1.1 2023"

Commit message: Ordered Version 1.0
Other:
- board text added: "1"
- board text added: "6"
- board text added: "RJ12 BB v1.0 2023"
- board text removed: "RJ12 BB v1.1 2023"
Changed lines of the file:
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@@
   (gr_rect (start 93.98 69.723) (end 126.238 84.3534)
     (stroke (width 0.1) (type default)) (fill none) (layer "Edge.Cuts"))
-  (gr_text "RJ12 BB\nv1.1 2023" (at 107.0102 78.2066) (layer "B.SilkS")
+  (gr_text "RJ12 BB\nv1.0 2023" (at 106.8 77.4) (layer "B.SilkS")
     (effects (font (size 1 1) (thickness 0.15)) (justify left bottom mirror))
   )
-  (gr_text "5" (at 121.4628 81.788) (layer "F.SilkS")
+  (gr_text "2" (at 113.1 75.8) (layer "B.SilkS")
+    (effects (font (size 1 1) (thickness 0.15)) (justify left bottom mirror))
+  )
+  (gr_text "1" (at 114.5 74.6) (layer "B.SilkS")
+    (effects (font (size 1 1) (thickness 0.15)) (justify left bottom mirror))
+  )
+  (gr_text "5" (at 114.5 79.6) (layer "B.SilkS")
+    (effects (font (size 1 1) (thickness 0.15)) (justify left bottom mirror))
+  )
+  (gr_text "3" (at 114.5 77.1) (layer "B.SilkS")
+    (effects (font (size 1 1) (thickness 0.15)) (justify left bottom mirror))
+  )
+  (gr_text "6" (at 113.2 81) (layer "B.SilkS")
+    (effects (font (size 1 1) (thickness 0.15)) (justify left bottom mirror))
+  )
+  (gr_text "4" (at 113.2 78.4) (layer "B.SilkS")
+    (effects (font (size 1 1) (thickness 0.15)) (justify left bottom mirror))
+  )
+  (gr_text "5" (at 121.1 81.788) (layer "F.SilkS")
     (effects (font (size 1.5 1.5) (thickness 0.3) bold) (justify left bottom))
   )
-  (gr_text "4" (at 121.4628 73.9648) (layer "F.SilkS")
+  (gr_text "4" (at 121.1 73.9648) (layer "F.SilkS")
     (effects (font (size 1.5 1.5) (thickness 0.3) bold) (justify left bottom))
   )
-  (gr_text "3" (at 121.4628 76.572533) (layer "F.SilkS")
+  (gr_text "3" (at 121.1 76.572533) (layer "F.SilkS")
     (effects (font (size 1.5 1.5) (thickness 0.3) bold) (justify left bottom))
   )
-  (gr_text "2" (at 121.4628 79.180266) (layer "F.SilkS")
+  (gr_text "2" (at 121.1 79.180266) (layer "F.SilkS")
     (effects (font (size 1.5 1.5) (thickness 0.3) bold) (justify left bottom))
   )
